Commit message: Modificaciones de movimiento dentro de ROS2
Carpeta de carrito_prueba_description con modificaciones de movimiento dentro de ROS2, ejecutando comandos para su movimiento, tambien lanzando Rviz2 en segundo plano mientras solo se lanza Gazebo

File: carrito_prueba_description/urdf/carrito_prueba.xacro (robot description, xacro)
@@ -120,5 +120,5 @@
   <parent link="base_link"/>
   <child link="llanta_1_1"/>
-  <axis xyz="0.0 -1.0 0.0"/>
+  <axis xyz="0.0 1.0 0.0"/>
 </joint>
 <joint name="joint3" type="continuous">
@@ -132,5 +132,5 @@
   <parent link="base_link"/>
   <child link="llanta_4_1"/>
-  <axis xyz="0.0 -1.0 0.0"/>
+  <axis xyz="0.0 1.0 0.0"/>
 </joint>
 </robot>
